File: dmm_board/dmm_board.kicad_sch (KiCad schematic)
At the start: 0 parts

Commit message: do da eth phy
Other:
- added sheet analog (analog.kicad_sch)
- added sheet cpu (cpu.kicad_sch)
- added sheet ethernet (ethernet.kicad_sch)
- added sheet power_mech (power.kicad_sch)
