File: dmm_board/current_input.kicad_sch (KiCad schematic)
At the start: 11 parts

Commit message: stuff
Parts:
- removed K?: AZ850P1-x, Relay_THT:Relay_DPDT_FRT5, symbol good_things:AZ850P1-x
- added D?: 1N4007, Diode_THT:D_DO-41_SOD81_P7.62mm_Horizontal, symbol Device:D
- added D?: RSX301L-30TE25, good_things:SOD-106, symbol Device:D
- added K?: m4-12h, Relay_THT:Relay_DPDT_FRT5, symbol good_things:m4-12h
- added Q?: 2N7002P, Package_TO_SOT_SMD:SOT-23_Handsoldering, symbol Device:Q_NMOS_GSD
- added R?: 470, symbol Device:R
- R?: value 500 -> 100
- R?: value 5 -> 500m
Connections:
- net SHUNT_OUT: now also K?.8
- net at R?.1: now also K?.6
- net at R?.1: now also K?.7
- net at D?.2 (A), D?.2 (A): now also D?.1 (K); no longer D?.1 (K)
- new net: D?.1 (K), D?.2 (A)
- new net +12V: K?.10
- new net GND: D?.2 (A), Q?.2 (S)
- new net MA_RANGE: R?.2
- new net ma_ua_relay_coil: D?.1 (K), K?.1, Q?.3 (D)
- new net ma_ua_relay_gate: Q?.1 (G), R?.1
Other:
- note added: "3mm isolation is good enuf pcbway.com/project/question/Minimum_distance_between_traces_for_250_400VDC.html"
- note added: "conducts a lot if voltage over shunts are above 4*diode_drop or below -4*diode_drop Limits voltage to +-2.8V assuming Si diodes"
- note added: "measure reverse current of this setup 1n4007 should be sufficiently small at 2V forward voltage such that no error significant error is seen say <1uA maximum else add more diodes at 1.4V over diodes this gives 6uA. 1V over diodes give 430nA at 0.2V over diodes this gives 25uV over 100k that is 250pA usnig a 10x amp this should be good i guess."
- note removed: "conducts a lot if voltage over shunts are above 3*diode_drop or below -3*diode_drop Limits voltage to +-2.1V assuming Si diodes"
- note removed: "measure reverse current of this setup 1n4007 should be sufficiently small at 2V forward voltage such that no error significant error is seen say <1uA maximum else add more diodes"
- moved on the sheet: D?, F?, R?

Commit message: more analog input work
need new amp for current -8 instead of -9 that
-8 is unity gain stable -9 is not
Parts:
- removed D?: RSX301L-30TE25, good_things:SOD-106, symbol Device:D
- added D?: 1N4007, Diode_THT:D_DO-41_SOD81_P7.62mm_Horizontal, symbol Device:D
Connections:
- net GND: now also D?.2 (A)
- net ma_ua_relay_coil: now also D?.1 (K)
Changed lines of the file:
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@@
   (junction (at 98.425 97.155) (diameter 0) (color 0 0 0 0)
   )
+  (junction (at 189.865 38.1) (diameter 0) (color 0 0 0 0)
+  )
   (junction (at 202.565 106.045) (diameter 0) (color 0 0 0 0)
   )
   (junction (at 189.865 93.98) (diameter 0) (color 0 0 0 0)
   )
-  (junction (at 189.865 82.55) (diameter 0) (color 0 0 0 0)
-  )
   (wire (pts (xy 202.565 106.045) (xy 210.82 106.045))
     (stroke (width 0) (type default) (color 0 0 0 0))
@@
     (stroke (width 0) (type default) (color 0 0 0 0))
   )
-  (wire (pts (xy 189.865 82.55) (xy 189.865 93.98))
-    (stroke (width 0) (type default) (color 0 0 0 0))
-  )
   (wire (pts (xy 191.77 90.17) (xy 182.88 90.17))
     (stroke (width 0) (type default) (color 0 0 0 0))
@@
     (stroke (width 0) (type default) (color 0 0 0 0))
   )
+  (wire (pts (xy 189.865 38.1) (xy 189.865 93.98))
+    (stroke (width 0) (type default) (color 0 0 0 0))
+  )
   (wire (pts (xy 189.865 116.84) (xy 189.865 115.57))
     (stroke (width 0) (type default) (color 0 0 0 0))
   )
-  (wire (pts (xy 189.865 82.55) (xy 264.795 82.55))
+  (wire (pts (xy 189.865 38.1) (xy 264.795 38.1))
     (stroke (width 0) (type default) (color 0 0 0 0))
   )
@@
     (stroke (width 0) (type default) (color 0 0 0 0))
   )
-  (wire (pts (xy 189.865 38.1) (xy 189.865 82.55))
-    (stroke (width 0) (type default) (color 0 0 0 0))
-  )
   (wire (pts (xy 153.035 88.265) (xy 153.035 97.155))
     (stroke (width 0) (type default) (color 0 0 0 0))
@@
     (stroke (width 0) (type default) (color 0 0 0 0))
   )
-  (wire (pts (xy 189.865 122.555) (xy 233.045 122.555))
+  (wire (pts (xy 189.865 122.555) (xy 264.795 122.555))
     (stroke (width 0) (type default) (color 0 0 0 0))
   )
@@
     (effects (font (size 1.27 1.27)) (justify left))
   )
-  (hierarchical_label "COM_OUT" (shape input) (at 233.045 122.555 0)
+  (hierarchical_label "COM_OUT" (shape input) (at 264.795 122.555 0)
     (effects (font (size 1.27 1.27)) (justify left))
   )
@@
     (effects (font (size 1.27 1.27)) (justify right))
   )
-  (hierarchical_label "SHUNT_OUT" (shape input) (at 264.795 82.55 0)
+  (hierarchical_label "SHUNT_OUT" (shape input) (at 264.795 38.1 0)
     (effects (font (size 1.27 1.27)) (justify left))
   )
@@
     (pin "2")
   )
-  (symbol (lib_id "Device:D") (at 193.675 64.77 270) (unit 1)
-    (in_bom yes) (on_board yes) (fields_autoplaced)
-    (property "Reference" "D?" (id 0) (at 195.707 63.8615 90)
-      (effects (font (size 1.27 1.27)) (justify left))
-    )
-    (property "Value" "RSX301L-30TE25" (id 1) (at 195.707 66.6366 90)
-      (effects (font (size 1.27 1.27)) (justify left))
-    )
-    (property "Footprint" "good_things:SOD-106" (id 2) (at 193.675 64.77 0)
-      (effects (font (size 1.27 1.27)) hide)
-    )
-    (property "Datasheet" "~" (id 3) (at 193.675 64.77 0)
-      (effects (font (size 1.27 1.27)) hide)
-    )
-    (pin "1")
-    (pin "2")
-  )
   (symbol (lib_id "Device:R") (at 153.035 84.455 0) (unit 1)
     (in_bom yes) (on_board yes) (fields_autoplaced)
@@
       (effects (font (size 1.27 1.27)) hide)
     )
+    (pin "1")
+    (pin "2")
+  )
+  (symbol (lib_id "Device:D") (at 193.675 64.77 270) (unit 1)
+    (in_bom yes) (on_board yes) (fields_autoplaced)
+    (property "Reference" "D?" (id 0) (at 195.707 63.8615 90)
+      (effects (font (size 1.27 1.27)) (justify left))
+    )
+    (property "Value" "1N4007" (id 1) (at 195.707 66.6366 90)
+      (effects (font (size 1.27 1.27)) (justify left))
+    )
+    (property "Footprint" "Diode_THT:D_DO-41_SOD81_P7.62mm_Horizontal" (id 2) (at 193.675 64.77 0)
+      (effects (font (size 1.27 1.27)) hide)
+    )
+    (property "Datasheet" "~" (id 3) (at 193.675 64.77 0)
+      (effects (font (size 1.27 1.27)) hide)
+    )
